Commit message: jumps off

File: platform.urdf (robot description, URDF)
Before this commit: robot platform, 1 links, 0 joints
Links:
- link p: geometry collision box size=4 4 0.1; visual box size=4 4 0.1

Commit message: gliding

File: platform.urdf (robot description, URDF)
Before this commit: robot platform, 1 links, 0 joints
Links:
- link p: geometry collision box size=3.5 4 0.1; visual box size=3.5 4 0.1
