Commit message: finished slide 11

File: body.urdf (robot description, URDF)
Before this commit: robot robot, 2 links, 1 joints
Links:
- removed link Leg
- removed link Torso
- added link Link0, mass 1; collision box size=1 1 1; visual box size=1 1 1
- added link Link1, mass 1; collision box size=1 1 1; visual box size=1 1 1
- added link Link2, mass 1; collision box size=1 1 1; visual box size=1 1 1
- added link Link3, mass 1; collision box size=1 1 1; visual box size=1 1 1
- added link Link4, mass 1; collision box size=1 1 1; visual box size=1 1 1
Joints:
- removed joint Torso_Leg
- added joint Link0_Link1: type revolute, parent Link0, child Link1, origin xyz=0 0 1 rpy=0 0 0, axis 0 1 0, limit lower=-3.14159 upper=3.14159 effort=0.0 velocity=0.0
- added joint Link1_Link2: type revolute, parent Link1, child Link2, origin xyz=0 0 1 rpy=0 0 0, axis 0 1 0, limit lower=-3.14159 upper=3.14159 effort=0.0 velocity=0.0
- added joint Link2_Link3: type revolute, parent Link2, child Link3, origin xyz=0 0.5 0.5 rpy=0 0 0, axis 0 1 0, limit lower=-3.14159 upper=3.14159 effort=0.0 velocity=0.0
- added joint Link3_Link4: type revolute, parent Link3, child Link4, origin xyz=0 1 0 rpy=0 0 0, axis 0 1 0, limit lower=-3.14159 upper=3.14159 effort=0.0 velocity=0.0

Commit message: joints

File: body.urdf (robot description, URDF)
Before this commit: robot robot, 5 links, 4 joints
Links:
- removed link Link0
- removed link Link1
- removed link Link2
- removed link Link3
- removed link Link4
- added link BackLeg, mass 1; collision box size=1 1 1; visual box size=1 1 1
- added link FrontLeg, mass 1; collision box size=1 1 1; visual box size=1 1 1
- added link Torso, mass 1; collision box size=1 1 1; visual box size=1 1 1
Joints:
- removed joint Link0_Link1
- removed joint Link1_Link2
- removed joint Link2_Link3
- removed joint Link3_Link4
- added joint BackLeg_Torso: type revolute, parent BackLeg, child Torso, origin xyz=1 0 1 rpy=0 0 0, axis 0 1 0, limit lower=-3.14159 upper=3.14159 effort=0.0 velocity=0.0
- added joint Torso_FrontLeg: type revolute, parent Torso, child FrontLeg, origin xyz=1 0 0 rpy=0 0 0, axis 0 1 0, limit lower=-3.14159 upper=3.14159 effort=0.0 velocity=0.0

Commit message: sensors finished + edited

File: body.urdf (robot description, URDF)
Before this commit: robot robot, 3 links, 2 joints
Joints:
- removed joint BackLeg_Torso
- added joint Torso_BackLeg: type revolute, parent Torso, child BackLeg, origin xyz=-0.5 0 1 rpy=0 0 0, axis 0 1 0, limit lower=-3.14159 upper=3.14159 effort=0.0 velocity=0.0
- joint Torso_FrontLeg: origin xyz=1 0 0 rpy=0 0 0 -> xyz=0.5 0 1 rpy=0 0 0

Commit message: finished Changing joint axes tentatively

File: body.urdf (robot description, URDF)
Before this commit: robot robot, 3 links, 2 joints
Links:
- link BackLeg: geometry collision box size=0.2 1 0.2; visual box size=0.2 1 0.2
- link FrontLeg: geometry collision box size=0.2 1 0.2; visual box size=0.2 1 0.2
Joints:
- joint Torso_BackLeg: axis 0 1 0 -> 1.5 0 0; origin xyz=-0.5 0 1 rpy=0 0 0 -> xyz=0 -0.5 1 rpy=0 0 0
- joint Torso_FrontLeg: axis 0 1 0 -> 1 0 0; origin xyz=0.5 0 1 rpy=0 0 0 -> xyz=0 0.5 1 rpy=0 0 0

Commit message: added four top legs

File: body.urdf (robot description, URDF)
Before this commit: robot robot, 3 links, 2 joints
Links:
- added link LeftLeg, mass 1; collision box size=1 0.2 0.2; visual box size=1 0.2 0.2
- added link RightLeg, mass 1; collision box size=1 0.2 0.2; visual box size=1 0.2 0.2
Joints:
- added joint Torso_LeftLeg: type revolute, parent Torso, child LeftLeg, origin xyz=-0.5 0 1 rpy=0 0 0, axis 0 1 0, limit lower=-3.14159 upper=3.14159 effort=0.0 velocity=0.0
- added joint Torso_RightLeg: type revolute, parent Torso, child RightLeg, origin xyz=0.5 0 1 rpy=0 0 0, axis 0 1 0, limit lower=-3.14159 upper=3.14159 effort=0.0 velocity=0.0
- joint Torso_BackLeg: axis 1.5 0 0 -> 1 0 0

Commit message: got quad body set up

File: body.urdf (robot description, URDF)
Before this commit: robot robot, 5 links, 4 joints
Links:
- added link BackLegLow, mass 1; collision box size=0.2 0.2 1; visual box size=0.2 0.2 1
- added link FrontLegLow, mass 1; collision box size=0.2 0.2 1; visual box size=0.2 0.2 1
- added link LeftLegLow, mass 1; collision box size=0.2 0.2 1; visual box size=0.2 0.2 1
- added link RightLegLow, mass 1; collision box size=0.2 0.2 1; visual box size=0.2 0.2 1
Joints:
- added joint BackLeg_BackLegLow: type revolute, parent BackLeg, child BackLegLow, origin xyz=0 -1 0 rpy=0 0 0, axis 1 0 0, limit lower=-3.14159 upper=3.14159 effort=0.0 velocity=0.0
- added joint FrontLeg_FrontLegLow: type revolute, parent FrontLeg, child FrontLegLow, origin xyz=0 1 0 rpy=0 0 0, axis 1 0 0, limit lower=-3.14159 upper=3.14159 effort=0.0 velocity=0.0
- added joint LeftLeg_LeftLegLow: type revolute, parent LeftLeg, child LeftLegLow, origin xyz=-1 0 0 rpy=0 0 0, axis 0 1 0, limit lower=-3.14159 upper=3.14159 effort=0.0 velocity=0.0
- added joint RightLeg_RightLegLow: type revolute, parent RightLeg, child RightLegLow, origin xyz=1 0 0 rpy=0 0 0, axis 0 1 0, limit lower=-3.14159 upper=3.14159 effort=0.0 velocity=0.0

Commit message: got prelim force stuff down

File: body.urdf (robot description, URDF)
Before this commit: robot robot, 9 links, 8 joints
Links:
- added link LeftEndWing, mass 1; collision box size=0.75 1 0.05; visual box size=0.75 1 0.05
- added link LeftUpperWing, mass 1; collision box size=1 1 0.05; visual box size=1 1 0.05
- added link RightEndWing, mass 1; collision box size=0.75 1 0.05; visual box size=0.75 1 0.05
- added link RightUpperWing, mass 1; collision box size=1 1 0.05; visual box size=1 1 0.05
- link Torso: geometry collision box size=1 1 1.5; visual box size=1 1 1.5
Joints:
- added joint LeftUpperWing_LeftEndWing: type revolute, parent LeftUpperWing, child LeftEndWing, origin xyz=0 0.5 0 rpy=0 0 0, axis 0 1 0, limit lower=-3.14159 upper=3.14159 effort=0.0 velocity=0.0
- added joint RightUpperWing_RightEndWing: type revolute, parent RightUpperWing, child RightEndWing, origin xyz=0 -0.5 0 rpy=0 0 0, axis 0 1 0, limit lower=-3.14159 upper=3.14159 effort=0.0 velocity=0.0
- added joint Torso_LeftUpperWing: type revolute, parent Torso, child LeftUpperWing, origin xyz=0 0.5 5.5 rpy=0 0 0, axis 0 1 0, limit lower=-3.14159 upper=3.14159 effort=0.0 velocity=0.0
- added joint Torso_RightUpperWing: type revolute, parent Torso, child RightUpperWing, origin xyz=0 -0.5 5.5 rpy=0 0 0, axis 0 1 0, limit lower=-3.14159 upper=3.14159 effort=0.0 velocity=0.0
- joint Torso_BackLeg: origin xyz=0 -0.5 1 rpy=0 0 0 -> xyz=0 -0.5 5 rpy=0 0 0
- joint Torso_FrontLeg: origin xyz=0 0.5 1 rpy=0 0 0 -> xyz=0 0.5 5 rpy=0 0 0
- joint Torso_LeftLeg: origin xyz=-0.5 0 1 rpy=0 0 0 -> xyz=-0.5 0 5 rpy=0 0 0
- joint Torso_RightLeg: origin xyz=0.5 0 1 rpy=0 0 0 -> xyz=0.5 0 5 rpy=0 0 0

Commit message: jumping?

File: body.urdf (robot description, URDF)
Before this commit: robot robot, 13 links, 12 joints
Links:
- link LeftEndWing: geometry collision box size=1 1 0.01; visual box size=1 1 0.01
- link LeftUpperWing: geometry collision box size=1.5 1.25 0.01; visual box size=1.5 1.25 0.01
- link RightEndWing: geometry collision box size=1 1 0.01; visual box size=1 1 0.01
- link RightUpperWing: geometry collision box size=1.5 1.25 0.01; visual box size=1.5 1.25 0.01
- link Torso: geometry collision box size=1 1 1; visual box size=1 1 1

Commit message: goes flying... adjust the drag

File: body.urdf (robot description, URDF)
Before this commit: robot robot, 13 links, 12 joints
Joints:
- joint Torso_BackLeg: origin xyz=0 -0.5 5 rpy=0 0 0 -> xyz=0 -0.5 9 rpy=0 0 0
- joint Torso_FrontLeg: origin xyz=0 0.5 5 rpy=0 0 0 -> xyz=0 0.5 9 rpy=0 0 0
- joint Torso_LeftLeg: origin xyz=-0.5 0 5 rpy=0 0 0 -> xyz=-0.5 0 9 rpy=0 0 0
- joint Torso_LeftUpperWing: origin xyz=0 0.5 5.5 rpy=0 0 0 -> xyz=0 0.5 9.5 rpy=0 0 0
- joint Torso_RightLeg: origin xyz=0.5 0 5 rpy=0 0 0 -> xyz=0.5 0 9 rpy=0 0 0
- joint Torso_RightUpperWing: origin xyz=0 -0.5 5.5 rpy=0 0 0 -> xyz=0 -0.5 9.5 rpy=0 0 0

File: platform.urdf (robot description, URDF)
Before this commit: robot platform, 1 links, 0 joints
Links:
- link p: geometry collision box size=3.5 3.5 0.1; visual box size=3.5 3.5 0.1

Commit message: dragonfly body

File: body.urdf (robot description, URDF)
Before this commit: robot robot, 13 links, 12 joints
Links:
- removed link LeftEndWing
- removed link LeftUpperWing
- removed link RightEndWing
- removed link RightUpperWing
- added link Head, mass 1; collision box size=1.5 1.5 1.5; visual box size=1.5 1.5 1.5
- added link LeftBackWing, mass 1; collision box size=0.75 3 0.01; visual box size=0.75 3 0.01
- added link LeftFrontWing, mass 1; collision box size=0.5 3 0.01; visual box size=0.5 3 0.01
- added link RightBackWing, mass 1; collision box size=0.75 3 0.01; visual box size=0.75 3 0.01
- added link RightFrontWing, mass 1; collision box size=0.5 3 0.01; visual box size=0.5 3 0.01
- link Torso: geometry collision box size=4 0.75 1; visual box size=4 0.75 1
Joints:
- removed joint LeftUpperWing_LeftEndWing
- removed joint RightUpperWing_RightEndWing
- removed joint Torso_LeftUpperWing
- removed joint Torso_RightUpperWing
- added joint Torso_Head: type revolute, parent Torso, child Head, origin xyz=0 4 9 rpy=0 0 0, axis 1 0 0, limit lower=-3.14159 upper=3.14159 effort=0.0 velocity=0.0
- added joint Torso_LeftBackWing: type revolute, parent Torso, child LeftBackWing, origin xyz=-0.25 -1 9.5 rpy=0 0 0, axis 0 1 0, limit lower=-3.14159 upper=3.14159 effort=0.0 velocity=0.0
- added joint Torso_LeftFrontWing: type revolute, parent Torso, child LeftFrontWing, origin xyz=0.25 -1 9.5 rpy=0 0 0, axis 0 1 0, limit lower=-3.14159 upper=3.14159 effort=0.0 velocity=0.0
- added joint Torso_RightBackWing: type revolute, parent Torso, child RightBackWing, origin xyz=-0.25 0 9.5 rpy=0 0 0, axis 0 1 0, limit lower=-3.14159 upper=3.14159 effort=0.0 velocity=0.0
- added joint Torso_RightFrontWing: type revolute, parent Torso, child RightFrontWing, origin xyz=0.25 0 9.5 rpy=0 0 0, axis 0 1 0, limit lower=-3.14159 upper=3.14159 effort=0.0 velocity=0.0

Commit message: dragonfly save values

File: body.urdf (robot description, URDF)
Before this commit: robot robot, 14 links, 13 joints
Links:
- link Head: geometry collision box size=1 1.5 1; visual box size=1 1.5 1
- link Torso: geometry collision box size=5 0.5 0.5; visual box size=5 0.5 0.5
Joints:
- joint Torso_Head: origin xyz=0 4 9 rpy=0 0 0 -> xyz=-0.5 4 9 rpy=0 0 0
- joint Torso_LeftBackWing: origin xyz=-0.25 -1 9.5 rpy=0 0 0 -> xyz=-0.25 -1 9 rpy=0 0 0
- joint Torso_LeftFrontWing: origin xyz=0.25 -1 9.5 rpy=0 0 0 -> xyz=0.25 -1 9 rpy=0 0 0
- joint Torso_RightBackWing: origin xyz=-0.25 0 9.5 rpy=0 0 0 -> xyz=-0.25 0 9 rpy=0 0 0
- joint Torso_RightFrontWing: origin xyz=0.25 0 9.5 rpy=0 0 0 -> xyz=0.25 0 9 rpy=0 0 0

Commit message: working

File: body.urdf (robot description, URDF)
Before this commit: robot robot, 14 links, 13 joints
Links:
- removed link Head
- removed link LeftBackWing
- removed link LeftFrontWing
- removed link RightBackWing
- removed link RightFrontWing
- added link LeftEndWing, mass 1; collision box size=1 1 0.01; visual box size=1 1 0.01
- added link LeftUpperWing, mass 1; collision box size=1.5 1.25 0.01; visual box size=1.5 1.25 0.01
- added link RightEndWing, mass 1; collision box size=1 1 0.01; visual box size=1 1 0.01
- added link RightUpperWing, mass 1; collision box size=1.5 1.25 0.01; visual box size=1.5 1.25 0.01
- link Torso: geometry collision box size=1 1 1; visual box size=1 1 1
Joints:
- removed joint Torso_Head
- removed joint Torso_LeftBackWing
- removed joint Torso_LeftFrontWing
- removed joint Torso_RightBackWing
- removed joint Torso_RightFrontWing
- added joint LeftUpperWing_LeftEndWing: type revolute, parent LeftUpperWing, child LeftEndWing, origin xyz=0 0.5 0 rpy=0 0 0, axis 0 1 0, limit lower=-3.14159 upper=3.14159 effort=0.0 velocity=0.0
- added joint RightUpperWing_RightEndWing: type revolute, parent RightUpperWing, child RightEndWing, origin xyz=0 -0.5 0 rpy=0 0 0, axis 0 1 0, limit lower=-3.14159 upper=3.14159 effort=0.0 velocity=0.0
- added joint Torso_LeftUpperWing: type revolute, parent Torso, child LeftUpperWing, origin xyz=0 0.5 9.5 rpy=0 0 0, axis 0 1 0, limit lower=-3.14159 upper=3.14159 effort=0.0 velocity=0.0
- added joint Torso_RightUpperWing: type revolute, parent Torso, child RightUpperWing, origin xyz=0 -0.5 9.5 rpy=0 0 0, axis 0 1 0, limit lower=-3.14159 upper=3.14159 effort=0.0 velocity=0.0

Commit message: removed wings and put it back on floor

File: body.urdf (robot description, URDF)
Before this commit: robot robot, 13 links, 12 joints
Links:
- removed link LeftEndWing
- removed link LeftUpperWing
- removed link RightEndWing
- removed link RightUpperWing
Joints:
- removed joint LeftUpperWing_LeftEndWing
- removed joint RightUpperWing_RightEndWing
- removed joint Torso_LeftUpperWing
- removed joint Torso_RightUpperWing
- joint Torso_BackLeg: origin xyz=0 -0.5 9 rpy=0 0 0 -> xyz=0 -0.5 1 rpy=0 0 0
- joint Torso_FrontLeg: origin xyz=0 0.5 9 rpy=0 0 0 -> xyz=0 0.5 1 rpy=0 0 0
- joint Torso_LeftLeg: origin xyz=-0.5 0 9 rpy=0 0 0 -> xyz=-0.5 0 1 rpy=0 0 0
- joint Torso_RightLeg: origin xyz=0.5 0 9 rpy=0 0 0 -> xyz=0.5 0 1 rpy=0 0 0

Commit message: made torso longer and put legs on the sides

File: body.urdf (robot description, URDF)
Before this commit: robot robot, 9 links, 8 joints
Links:
- link LeftLeg: geometry collision box size=0.2 1 0.2; visual box size=0.2 1 0.2
- link RightLeg: geometry collision box size=0.2 1 0.2; visual box size=0.2 1 0.2
- link Torso: geometry collision box size=2 1 1; visual box size=2 1 1
Joints:
- joint LeftLeg_LeftLegLow: axis 0 1 0 -> 1 0 0; origin xyz=-1 0 0 rpy=0 0 0 -> xyz=0 -1 0 rpy=0 0 0
- joint RightLeg_RightLegLow: axis 0 1 0 -> 1 0 0; origin xyz=1 0 0 rpy=0 0 0 -> xyz=0 1 0 rpy=0 0 0
- joint Torso_LeftLeg: axis 0 1 0 -> 1 0 0; origin xyz=-0.5 0 1 rpy=0 0 0 -> xyz=0 -0.5 1 rpy=0 0 0
- joint Torso_RightLeg: axis 0 1 0 -> 1 0 0; origin xyz=0.5 0 1 rpy=0 0 0 -> xyz=0 0.5 1 rpy=0 0 0

Commit message: added head and legs, need to turn legs

File: body.urdf (robot description, URDF)
Before this commit: robot robot, 9 links, 8 joints
Links:
- added link Head, mass 1; collision box size=1 0.5 0.5; visual box size=1 0.5 0.5
- added link Neck, mass 1; collision box size=0.2 0.2 0.5; visual box size=0.2 0.2 0.5
- link Torso: geometry collision box size=2.25 1 0.5; visual box size=2.25 1 0.5
Joints:
- added joint Neck_Head: type revolute, parent Neck, child Head, origin xyz=0.25 0 0 rpy=0 0 0, axis 0 1 0, limit lower=-3.14159 upper=3.14159 effort=0.0 velocity=0.0
- added joint Torso_Neck: type revolute, parent Torso, child Neck, origin xyz=0.75 0 1 rpy=0 0 0, axis 0 1 0, limit lower=-3.14159 upper=3.14159 effort=0.0 velocity=0.0
- joint BackLeg_BackLegLow: axis 1 0 0 -> 0 1 0

Commit message: got 2 legs down

File: body.urdf (robot description, URDF)
Before this commit: robot robot, 11 links, 10 joints
Links:
- added link Thigh, mass 1; collision box size=0.2 0.5 0.2; visual box size=0.2 0.5 0.2
- added link ThighFront, mass 1; collision box size=0.2 0.5 0.2; visual box size=0.2 0.5 0.2
- link BackLeg: geometry collision box size=1 0.2 0.2; visual box size=1 0.2 0.2
- link FrontLeg: geometry collision box size=1 0.2 0.2; visual box size=1 0.2 0.2
Joints:
- removed joint Torso_BackLeg
- removed joint Torso_FrontLeg
- added joint ThighFront_FrontLeg: type revolute, parent ThighFront, child FrontLeg, origin xyz=0 0.5 0.5 rpy=0 0 0, axis 1 0 0, limit lower=-3.14159 upper=3.14159 effort=0.0 velocity=0.0
- added joint Thigh_BackLeg: type revolute, parent Thigh, child BackLeg, origin xyz=-0.5 -0.5 0.5 rpy=0 0 0, axis 0 1 0, limit lower=-3.14159 upper=3.14159 effort=0.0 velocity=0.0
- added joint Torso_Thigh: type revolute, parent Torso, child Thigh, origin xyz=0 -0.2 1 rpy=0 0 0, axis 0 1 0, limit lower=-3.14159 upper=3.14159 effort=0.0 velocity=0.0
- added joint Torso_ThighFront: type revolute, parent Torso, child ThighFront, origin xyz=0 0.2 1 rpy=0 0 0, axis 0 1 0, limit lower=-3.14159 upper=3.14159 effort=0.0 velocity=0.0
- joint BackLeg_BackLegLow: origin xyz=0 -1 0 rpy=0 0 0 -> xyz=-1 0 0 rpy=0 0 0
- joint FrontLeg_FrontLegLow: axis 1 0 0 -> 0 1 0; origin xyz=0 1 0 rpy=0 0 0 -> xyz=-0.5 0 0 rpy=0 0 0
- joint LeftLeg_LeftLegLow: axis 1 0 0 -> 0 1 0
- joint RightLeg_RightLegLow: axis 1 0 0 -> 0 1 0

Commit message: done for now

File: body.urdf (robot description, URDF)
Before this commit: robot robot, 13 links, 12 joints
Links:
- added link ThighLeft, mass 1; collision box size=0.2 0.5 0.2; visual box size=0.2 0.5 0.2
- added link ThighRight, mass 1; collision box size=0.2 0.5 0.2; visual box size=0.2 0.5 0.2
- link BackLeg: geometry collision box size=0.5 0.2 0.2; visual box size=0.5 0.2 0.2
- link FrontLeg: geometry collision box size=0.5 0.2 0.2; visual box size=0.5 0.2 0.2
- link LeftLeg: geometry collision box size=0.5 0.2 0.2; visual box size=0.5 0.2 0.2
- link RightLeg: geometry collision box size=0.5 0.2 0.2; visual box size=0.5 0.2 0.2
- link Torso: geometry collision box size=2 1 0.5; visual box size=2 1 0.5
Joints:
- removed joint Torso_LeftLeg
- removed joint Torso_RightLeg
- added joint ThighLeft_LeftLeg: type revolute, parent ThighLeft, child LeftLeg, origin xyz=0 -0.5 0 rpy=0 0 0, axis 0 1 0, limit lower=-3.14159 upper=3.14159 effort=0.0 velocity=0.0
- added joint ThighRight_RightLeg: type revolute, parent ThighRight, child RightLeg, origin xyz=0 0.5 0 rpy=0 0 0, axis 0 1 0, limit lower=-3.14159 upper=3.14159 effort=0.0 velocity=0.0
- added joint Torso_ThighLeft: type fixed, parent Torso, child ThighLeft, origin xyz=0.75 -0.2 1 rpy=0 0 0, axis 0 1 0, limit lower=-3.14159 upper=3.14159 effort=0.0 velocity=0.0
- added joint Torso_ThighRight: type fixed, parent Torso, child ThighRight, origin xyz=-0.75 0.2 1 rpy=0 0 0, axis 0 1 0, limit lower=-3.14159 upper=3.14159 effort=0.0 velocity=0.0
- joint BackLeg_BackLegLow: origin xyz=-1 0 0 rpy=0 0 0 -> xyz=-0.5 0 0 rpy=0 0 0
- joint LeftLeg_LeftLegLow: origin xyz=0 -1 0 rpy=0 0 0 -> xyz=-0.5 0 0 rpy=0 0 0
- joint Neck_Head: origin xyz=0.25 0 0 rpy=0 0 0 -> xyz=0 0 0.5 rpy=0 0 0; type revolute -> fixed
- joint RightLeg_RightLegLow: origin xyz=0 1 0 rpy=0 0 0 -> xyz=-0.5 0 0 rpy=0 0 0
- joint ThighFront_FrontLeg: axis 1 0 0 -> 0 1 0; origin xyz=0 0.5 0.5 rpy=0 0 0 -> xyz=0 0.5 0 rpy=0 0 0
- joint Thigh_BackLeg: origin xyz=-0.5 -0.5 0.5 rpy=0 0 0 -> xyz=0 -0.5 0 rpy=0 0 0
- joint Torso_Thigh: origin xyz=0 -0.2 1 rpy=0 0 0 -> xyz=-0.75 -0.2 1 rpy=0 0 0; type revolute -> fixed
- joint Torso_ThighFront: origin xyz=0 0.2 1 rpy=0 0 0 -> xyz=0.75 0.2 1 rpy=0 0 0; type revolute -> fixed

Commit message: adding hidden

File: body.urdf (robot description, URDF)
Before this commit: robot robot, 15 links, 14 joints
Links:
- added link TorsoSensor, mass 1; collision box size=1 0.01 0.4; visual box size=1 0.01 0.4
Joints:
- added joint Torso_TorsoSensor: type fixed, parent Torso, child TorsoSensor, origin xyz=0 0 0.5 rpy=0 0 0, axis 0 1 0, limit lower=-3.14159 upper=3.14159 effort=0.0 velocity=0.0
